File: pcb_v11/afterglow_pico.kicad_pcb (KiCad board)
At the start: 2 copper layers, 57.5 x 57.5 mm, 40 parts, among them J1 Conn_02x17_Odd_Even, J2 Conn_02x17_Odd_Even, U1 74LS21, U2 7408, U3 SN74LVC245AN, U4 SN74LVC245AN, U5 SC0915, U6 74LS245, U7 74LS245, U8 74LS157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

Commit message: PCB v1.2 preparations
Parts:
- R4: value 10k -> 4.7k
- U8, U9: value 74LS157 -> 74LS257
- moved AG_LOGO 0.20 mm to (199.8, 114.8)
- renumbered G*** to AG_LOGO, G*** to BFL_LOGO
Connections:
- R4 pad 1: GND -> /PICO_OUT_EN
- R4 pad 2: /PICO_OUT_EN -> GND
- R5 pad 1: Net-(R5-Pad1) -> /PICO_EN_OUT
- U3 pad 19: GND -> /PICO_EN_OUT
- U4 pad 19: GND -> /PICO_EN_OUT
- U5 pad 17: Net-(R5-Pad1) -> /PICO_EN_OUT
- U6 pad 19: Net-(R5-Pad1) -> /PICO_EN_OUT
- U7 pad 19: Net-(R5-Pad1) -> /PICO_EN_OUT
- U8 pad 15: Net-(R16-Pad2) -> /PICO_EN_OUT
- U9 pad 15: Net-(R16-Pad2) -> /PICO_EN_OUT
Routing:
- net GND: track 423.2 -> 0.00 mm, vias 8 -> 0
- net +5V: track 240.5 -> 0.00 mm, vias 6 -> 0
- net +3V3: track 164.3 -> 0.00 mm, vias 4 -> 0
- net /P33: track 94.4 -> 0.00 mm
- net /DIS3: track 86.8 -> 0.00 mm
- net /LROW_PICO: track 84.5 -> 0.00 mm, vias 2 -> 0
- net Net-(R16-Pad2): track 78.5 -> 0.00 mm, vias 3 -> 0
- net /PICO_BLANK: track 76.2 -> 0.00 mm, vias 1 -> 0
- net Net-(U5-Pad20): track 74.4 -> 0.00 mm, vias 1 -> 0
- net Net-(U5-Pad22): track 73.2 -> 0.00 mm, vias 3 -> 0
- net /D4: track 68.2 -> 0.00 mm, vias 4 -> 0
- net /OUT_SEL: track 64.3 -> 0.00 mm, vias 3 -> 0
- net /BLANK: track 58.9 -> 0.00 mm, vias 3 -> 0
- net /DIS1: track 58.8 -> 0.00 mm
- net /TRIAC: track 56.3 -> 0.00 mm, vias 3 -> 0
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Other:
- board text added: "74LS257"
- board text added: "74LVC245"
- board text added: "v1.2 WPC"
- board text removed: "74LS157"
