File: pcb_v13/afterglow_pico.kicad_pcb (KiCad board)
At the start: 4 copper layers, 69.4 x 88.1 mm, 88 parts, among them J1 USB_B_Micro, J2 Conn_01x02_Male, J3 Conn_01x02, J4 Conn_02x17_Odd_Even, J5 Conn_02x17_Odd_Even, U1 NCP1117-3.3_SOT223, U10 74HC257, U11 74HC257, U2 RP2040, U3 SN74LVC245AN, U4 SN74LVC245AN, U5 W25Q32JVSS, U6 74HC21, U7 7408, U8 74HC245, U9 74HC245, Y1 ABLS-12.000MHZ-B4-T

Commit message: Boettn
Parts:
- removed J3: Conn_01x02, Connector_PinHeader_2.54mm:PinHeader_1x02_P2.54mm_Vertical
- added SW1: SW_Push, Button_Switch_SMD:SW_SPST_B3U-1000P, F.Cu at (151.8, 63.1)
- moved R6 1.37 mm to (156.4, 63.0)
- renumbered PWR to PWR_LED1
Changed lines of the file:
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@@
     (property "Sheetname" "")
     (attr smd)
-    (fp_text reference "PWR" (at -2.635 -0.075) (layer "F.SilkS")
+    (fp_text reference "PWR_LED1" (at -2.635 -0.075) (layer "F.SilkS")
       (effects (font (size 1 1) (thickness 0.15)))
     )
@@
     )
   )
-  (footprint "Connector_PinHeader_2.54mm:PinHeader_1x02_P2.54mm_Vertical" (layer "F.Cu")
-    (at 152.72 61.65 -90)
-    (descr "Through hole straight pin header, 1x02, 2.54mm pitch, single row")
-    (tags "Through hole pin header THT 1x02 2.54mm single row")
-    (property "Sheetfile" "afterglow_pico.kicad_sch")
-    (property "Sheetname" "")
-    (attr through_hole)
-    (fp_text reference "J3" (at 2.725 1.045 180) (layer "F.SilkS")
-      (effects (font (size 1 1) (thickness 0.15)))
-    )
-    (fp_text value "Conn_01x02" (at 0 4.87 90) (layer "F.Fab")
-      (effects (font (size 1 1) (thickness 0.15)))
-    )
-    (fp_text user "${REFERENCE}" (at 0 1.27) (layer "F.Fab")
-      (effects (font (size 1 1) (thickness 0.15)))
-    )
-    (fp_line (start -1.33 1.27) (end 1.33 1.27) (layer "F.SilkS") (width 0.12))
-    (fp_line (start 1.33 1.27) (end 1.33 3.87) (layer "F.SilkS") (width 0.12))
-    (fp_line (start -1.33 0) (end -1.33 -1.33) (layer "F.SilkS") (width 0.12))
-    (fp_line (start -1.33 3.87) (end 1.33 3.87) (layer "F.SilkS") (width 0.12))
-    (fp_line (start -1.33 -1.33) (end 0 -1.33) (layer "F.SilkS") (width 0.12))
-    (fp_line (start -1.33 1.27) (end -1.33 3.87) (layer "F.SilkS") (width 0.12))
-    (fp_line (start 1.8 4.35) (end 1.8 -1.8) (layer "F.CrtYd") (width 0.05))
-    (fp_line (start -1.8 4.35) (end 1.8 4.35) (layer "F.CrtYd") (width 0.05))
-    (fp_line (start 1.8 -1.8) (end -1.8 -1.8) (layer "F.CrtYd") (width 0.05))
-    (fp_line (start -1.8 -1.8) (end -1.8 4.35) (layer "F.CrtYd") (width 0.05))
-    (fp_line (start 1.27 -1.27) (end 1.27 3.81) (layer "F.Fab") (width 0.1))
-    (fp_line (start -0.635 -1.27) (end 1.27 -1.27) (layer "F.Fab") (width 0.1))
-    (fp_line (start -1.27 -0.635) (end -0.635 -1.27) (layer "F.Fab") (width 0.1))
-    (fp_line (start 1.27 3.81) (end -1.27 3.81) (layer "F.Fab") (width 0.1))
-    (fp_line (start -1.27 3.81) (end -1.27 -0.635) (layer "F.Fab") (width 0.1))
-    (pad "1" thru_hole rect (at 0 0 270) (size 1.7 1.7) (drill 1) (layers *.Cu *.Mask)
-      (net 48 "/~{USB_BOOT}") (pinfunction "Pin_1") (pintype "passive"))
-    (pad "2" thru_hole oval (at 0 2.54 270) (size 1.7 1.7) (drill 1) (layers *.Cu *.Mask)
-      (net 1 "GND") (pinfunction "Pin_2") (pintype "passive"))
-    (model "${KICAD6_3DMODEL_DIR}/Connector_PinHeader_2.54mm.3dshapes/PinHeader_1x02_P2.54mm_Vertical.wrl"
-      (offset (xyz 0 0 0))
-      (scale (xyz 1 1 1))
-      (rotate (xyz 0 0 0))
-    )
-  )
   (footprint "Resistor_SMD:R_0402_1005Metric" (layer "F.Cu")
     (at 200.24 102.125 180)
@@
       (net 11 "/D4") (pintype "passive"))
     (model "${KICAD6_3DMODEL_DIR}/Resistor_SMD.3dshapes/R_0402_1005Metric.wrl"
+      (offset (xyz 0 0 0))
+      (scale (xyz 1 1 1))
+      (rotate (xyz 0 0 0))
+    )
+  )
+  (footprint "Button_Switch_SMD:SW_SPST_B3U-1000P" (layer "F.Cu")
+    (at 151.85 63.125)
+    (descr "Ultra-small-sized Tactile Switch with High Contact Reliability, Top-actuated Model, without Ground Terminal, without Boss")
+    (tags "Tactile Switch")
+    (property "Sheetfile" "afterglow_pico.kicad_sch")
+    (property "Sheetname" "")
+    (attr smd)
+    (fp_text reference "SW1" (at 0 -2.5) (layer "F.SilkS")
+      (effects (font (size 1 1) (thickness 0.15)))
+    )
+    (fp_text value "SW_Push" (at 0 2.5) (layer "F.Fab")
+      (effects (font (size 1 1) (thickness 0.15)))
+    )
+    (fp_text user "${REFERENCE}" (at 0 -2.5) (layer "F.Fab")
+      (effects (font (size 1 1) (thickness 0.15)))
+    )
+    (fp_line (start -1.65 -1.1) (end -1.65 -1.4) (layer "F.SilkS") (width 0.12))
+    (fp_line (start 1.65 -1.4) (end 1.65 -1.1) (layer "F.SilkS") (width 0.12))
+    (fp_line (start -1.65 1.4) (end 1.65 1.4) (layer "F.SilkS") (width 0.12))
+    (fp_line (start -1.65 1.1) (end -1.65 1.4) (layer "F.SilkS") (width 0.12))
+    (fp_line (start -1.65 -1.4) (end 1.65 -1.4) (layer "F.SilkS") (width 0.12))
+    (fp_line (start 1.65 1.4) (end 1.65 1.1) (layer "F.SilkS") (width 0.12))
+    (fp_line (start 2.4 1.65) (end 2.4 -1.65) (layer "F.CrtYd") (width 0.05))
+    (fp_line (start -2.4 1.65) (end 2.4 1.65) (layer "F.CrtYd") (width 0.05))
+    (fp_line (start -2.4 -1.65) (end -2.4 1.65) (layer "F.CrtYd") (width 0.05))
+    (fp_line (start 2.4 -1.65) (end -2.4 -1.65) (layer "F.CrtYd") (width 0.05))
+    (fp_line (start -1.5 -1.25) (end 1.5 -1.25) (layer "F.Fab") (width 0.1))
+    (fp_line (start -1.5 1.25) (end -1.5 -1.25) (layer "F.Fab") (width 0.1))
+    (fp_line (start 1.5 -1.25) (end 1.5 1.25) (layer "F.Fab") (width 0.1))
+    (fp_line (start 1.5 1.25) (end -1.5 1.25) (layer "F.Fab") (width 0.1))
+    (fp_circle (center 0 0) (end 0.75 0) (layer "F.Fab") (width 0.1) (fill none))
+    (pad "1" smd rect (at -1.7 0) (size 0.9 1.7) (layers "F.Cu" "F.Paste" "F.Mask")
+      (net 1 "GND") (pinfunction "1") (pintype "passive"))
+    (pad "2" smd rect (at 1.7 0) (size 0.9 1.7) (layers "F.Cu" "F.Paste" "F.Mask")
+      (net 48 "/~{USB_BOOT}") (pinfunction "2") (pintype "passive"))
+    (model "${KICAD6_3DMODEL_DIR}/Button_Switch_SMD.3dshapes/SW_SPST_B3U-1000P.wrl"
       (offset (xyz 0 0 0))
       (scale (xyz 1 1 1))
@@
   )
   (footprint "Resistor_SMD:R_0402_1005Metric" (layer "F.Cu")
-    (at 156.35 61.675 90)
+    (at 156.425 63.04 90)
     (descr "Resistor SMD 0402 (1005 Metric), square (rectangular) end terminal, IPC_7351 nominal, (Body size source: IPC-SM-782 page 72, https://www.pcb-3d.com/wordpress/wp-content/uploads/ipc-sm-782a_amendment_1_and_2.pdf), generated with kicad-footprint-generator")
     (tags "resistor")
