File: pcb_v13/afterglow_pico.kicad_sch (KiCad schematic)
At the start: 50 parts, among them J1 Conn_02x17_Odd_Even, J2 Conn_02x17_Odd_Even, J3 Conn_01x02_Male, U1 74LS21, U2 7408, U3 SN74LVC245AN, U4 SN74LVC245AN, U5 Raspberry Pi Pico, U6 74LS245, U7 74LS245, U8 74LS257, U9 74LS257

Commit message: Before routing
Parts:
- R1, R10, R11, R12, R13, R14, R15, R16, R17, R18, R19, R2, R20, R21, R22, R23, R24, R25, R26, R3, R4, R5, R6, R7, R8, R9: footprint Resistors_SMD:R_0805_HandSoldering -> pcb_v13:R_0805_HandSoldering

Commit message: PCB v1.3 progress
Parts:
- D1, D2: JLCPCB (none) -> C520634
- R17, R18, R19, R20, R21, R22, R23, R24: JLCPCB C17673 -> C17710
- R25: JLCPCB C17673 -> C4310
- R26: JLCPCB C17673 -> C17772
- U2: JLCPCB (none) -> C6802
- U5: JLCPCB (none) -> C5159530
Changed lines of the file:
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@@
       (effects (font (size 1.27 1.27)) (justify left bottom) hide)
+    )
+    (property "JLCPCB" "C5159530" (id 8) (at 153.67 69.85 0)
+      (effects (font (size 1.27 1.27)) hide)
     )
     (pin "1")
@@
       (effects (font (size 1.27 1.27)) hide)
     )
+    (property "JLCPCB" "C6802" (id 4) (at 127 151.13 0)
+      (effects (font (size 1.27 1.27)) hide)
+    )
     (pin "14")
     (pin "7")
@@
       (effects (font (size 1.27 1.27)) hide)
     )
+    (property "JLCPCB" "C6802" (id 4) (at 58.42 180.34 0)
+      (effects (font (size 1.27 1.27)) hide)
+    )
     (pin "14")
     (pin "7")
@@
       (effects (font (size 1.27 1.27)) hide)
     )
+    (property "JLCPCB" "C6802" (id 4) (at 86.36 177.8 0)
+      (effects (font (size 1.27 1.27)) hide)
+    )
     (pin "14")
     (pin "7")
@@
       (effects (font (size 1.27 1.27)) hide)
     )
-    (property "JLCPCB" "C17673" (id 4) (at 73.66 31.75 0)
+    (property "JLCPCB" "C17710" (id 4) (at 73.66 31.75 0)
       (effects (font (size 1.27 1.27)) hide)
     )
@@
       (effects (font (size 1.27 1.27)) hide)
     )
-    (property "JLCPCB" "C17673" (id 4) (at 78.74 89.535 0)
+    (property "JLCPCB" "C4310" (id 4) (at 78.74 89.535 0)
       (effects (font (size 1.27 1.27)) hide)
     )
@@
       (effects (font (size 1.27 1.27)) hide)
     )
-    (property "JLCPCB" "C17673" (id 4) (at 76.2 31.75 0)
+    (property "JLCPCB" "C17710" (id 4) (at 76.2 31.75 0)
       (effects (font (size 1.27 1.27)) hide)
     )
@@
       (effects (font (size 1.27 1.27)) hide)
     )
-    (property "JLCPCB" "C17673" (id 4) (at 78.74 31.75 0)
+    (property "JLCPCB" "C17710" (id 4) (at 78.74 31.75 0)
       (effects (font (size 1.27 1.27)) hide)
     )
@@
       (effects (font (size 1.27 1.27)) hide)
     )
-    (property "JLCPCB" "C17673" (id 4) (at 60.96 31.75 0)
+    (property "JLCPCB" "C17710" (id 4) (at 60.96 31.75 0)
       (effects (font (size 1.27 1.27)) hide)
     )
@@
       (effects (font (size 1.27 1.27)) hide)
     )
-    (property "JLCPCB" "C17673" (id 4) (at 68.58 31.75 0)
+    (property "JLCPCB" "C17710" (id 4) (at 68.58 31.75 0)
       (effects (font (size 1.27 1.27)) hide)
     )
@@
       (effects (font (size 1.27 1.27)) hide)
     )
-    (property "JLCPCB" "C17673" (id 4) (at 63.5 31.75 0)
+    (property "JLCPCB" "C17710" (id 4) (at 63.5 31.75 0)
       (effects (font (size 1.27 1.27)) hide)
     )
@@
     )
     (property "Datasheet" "https://www.infineon.com/dgdl/Infineon-BAT60ASERIES-DS-v01_01-en.pdf?fileId=db3a304313d846880113def70c9304a9" (id 3) (at 55.245 114.3 0)
+      (effects (font (size 1.27 1.27)) hide)
+    )
+    (property "JLCPCB" "C520634" (id 4) (at 55.245 114.3 0)
       (effects (font (size 1.27 1.27)) hide)
     )
@@
       (effects (font (size 1.27 1.27)) hide)
     )
+    (property "JLCPCB" "C520634" (id 4) (at 183.515 24.765 90)
+      (effects (font (size 1.27 1.27)) hide)
+    )
     (pin "1")
     (pin "2")
@@
       (effects (font (size 1.27 1.27)) hide)
     )
-    (property "JLCPCB" "C17673" (id 4) (at 71.12 31.75 0)
+    (property "JLCPCB" "C17710" (id 4) (at 71.12 31.75 0)
       (effects (font (size 1.27 1.27)) hide)
     )
@@
       (effects (font (size 1.27 1.27)) hide)
     )
-    (property "JLCPCB" "C17673" (id 4) (at 66.04 31.75 0)
+    (property "JLCPCB" "C17710" (id 4) (at 66.04 31.75 0)
       (effects (font (size 1.27 1.27)) hide)
     )
@@
       (effects (font (size 1.27 1.27)) hide)
     )
-    (property "JLCPCB" "C17673" (id 4) (at 81.28 89.535 0)
-      (effects (font (size 1.27 1.27)) hide)
-    )
+    (property "JLCPCB" "C17772" (id 4) (at 81.28 89.535 0)
+      (effects (font (size 1.27 1.27)) hide)
+    )

Commit message: First attempt
Parts:
- removed U5: Raspberry Pi Pico, SnapEDA Library:MODULE_SC0915, symbol SC0915:SC0915
- added C1, C2: 27p, Capacitor_SMD:C_0402_1005Metric, symbol Device:C
- added C10, C11, C12, C13, C14, C15, C18, C3, C5, C8: 100n, Capacitor_SMD:C_0402_1005Metric, symbol Device:C
- added C4, C7: 10u, Capacitor_SMD:C_0805_2012Metric, symbol Device:C
- added C6, C9: 1u, Capacitor_SMD:C_0402_1005Metric, symbol Device:C
- added D2: BAT60A, Diode_SMD:D_SOD-323, symbol Diode:BAT60A
- added D4: WS2812B, LED_SMD:LED_WS2812B_PLCC4_5.0x5.0mm_P3.2mm, symbol LED:WS2812B
- added J1: USB_B_Micro, Connector_USB:USB_Micro-B_Molex-105017-0001, symbol RP2040_minimal-rescue:USB_B_Micro-Connector
- added J3: Conn_01x02, Connector_PinHeader_2.54mm:PinHeader_1x02_P2.54mm_Vertical, symbol Connector_Generic:Conn_01x02
- added R1, R6: 1k, Resistor_SMD:R_0402_1005Metric, symbol Device:R
- added R14: 10k, Resistor_SMD:R_0402_1005Metric, symbol Device:R
- added R2, R3: 27, Resistor_SMD:R_0402_1005Metric, symbol Device:R
- added R32, R33, R34, R35, R36: 4.7k, Resistor_SMD:R_0402_1005Metric, symbol Device:R_Small
- added U1: NCP1117-3.3_SOT223, Package_TO_SOT_SMD:SOT-223-3_TabPin2, symbol Regulator_Linear:NCP1117-3.3_SOT223
- added U2: RP2040, RP2040_minimal:RP2040-QFN-56, symbol MCU_RaspberryPi_RP2040:RP2040
- added U5: W25Q32JVSS, Package_SO:SOIC-8_5.23x5.23mm_P1.27mm, symbol Memory_Flash:W25Q32JVSS
- added Y1: ABLS-12.000MHZ-B4-T, RP2040_minimal:Crystal_SMD_HC49-US, symbol Device:Crystal
- C16: renamed from C1; footprint Capacitors_SMD:C_0805_HandSoldering -> Capacitor_SMD:C_0402_1005Metric
- C17: renamed from C2; footprint Capacitors_SMD:C_0805_HandSoldering -> Capacitor_SMD:C_0402_1005Metric
- C19: renamed from C7; footprint Capacitors_SMD:C_0805_HandSoldering -> Capacitor_SMD:C_0402_1005Metric
- C20: renamed from C3; footprint Capacitors_SMD:C_0805_HandSoldering -> Capacitor_SMD:C_0402_1005Metric
- C21: renamed from C4; footprint Capacitors_SMD:C_0805_HandSoldering -> Capacitor_SMD:C_0402_1005Metric
- C22: renamed from C5; footprint Capacitors_SMD:C_0805_HandSoldering -> Capacitor_SMD:C_0402_1005Metric
- C23: renamed from C6; footprint Capacitors_SMD:C_0805_HandSoldering -> Capacitor_SMD:C_0402_1005Metric
- C24: renamed from C8; footprint Capacitors_SMD:C_0805_HandSoldering -> Capacitor_SMD:C_0402_1005Metric
- PWR_LED1: footprint LEDs:LED_0805_HandSoldering -> LED_SMD:LED_0402_1005Metric
- R10: renamed from R22; footprint pcb_v13:R_0805_HandSoldering -> Resistor_SMD:R_0402_1005Metric
- R11: renamed from R23; footprint pcb_v13:R_0805_HandSoldering -> Resistor_SMD:R_0402_1005Metric
- R12: renamed from R24; footprint pcb_v13:R_0805_HandSoldering -> Resistor_SMD:R_0402_1005Metric
- R13: renamed from R25; footprint pcb_v13:R_0805_HandSoldering -> Resistor_SMD:R_0402_1005Metric
- R15: renamed from R26; footprint pcb_v13:R_0805_HandSoldering -> Resistor_SMD:R_0402_1005Metric
- R16: renamed from R2; footprint pcb_v13:R_0805_HandSoldering -> Resistor_SMD:R_0402_1005Metric
- R17: renamed from R6; footprint pcb_v13:R_0805_HandSoldering -> Resistor_SMD:R_0402_1005Metric
- R18: renamed from R7; footprint pcb_v13:R_0805_HandSoldering -> Resistor_SMD:R_0402_1005Metric
- R19: renamed from R8; footprint pcb_v13:R_0805_HandSoldering -> Resistor_SMD:R_0402_1005Metric
- R20: renamed from R9; footprint pcb_v13:R_0805_HandSoldering -> Resistor_SMD:R_0402_1005Metric
- R21: renamed from R10; footprint pcb_v13:R_0805_HandSoldering -> Resistor_SMD:R_0402_1005Metric
- R22: renamed from R11; footprint pcb_v13:R_0805_HandSoldering -> Resistor_SMD:R_0402_1005Metric
- R23: renamed from R12; footprint pcb_v13:R_0805_HandSoldering -> Resistor_SMD:R_0402_1005Metric
- R24: renamed from R13; footprint pcb_v13:R_0805_HandSoldering -> Resistor_SMD:R_0402_1005Metric
- R25: renamed from R14; footprint pcb_v13:R_0805_HandSoldering -> Resistor_SMD:R_0402_1005Metric
- R26: renamed from R15; footprint pcb_v13:R_0805_HandSoldering -> Resistor_SMD:R_0402_1005Metric
- R27: renamed from R5; footprint pcb_v13:R_0805_HandSoldering -> Resistor_SMD:R_0402_1005Metric
- R28: renamed from R16; footprint pcb_v13:R_0805_HandSoldering -> Resistor_SMD:R_0402_1005Metric
- R29: renamed from R3; footprint pcb_v13:R_0805_HandSoldering -> Resistor_SMD:R_0402_1005Metric
- R30: renamed from R4; footprint pcb_v13:R_0805_HandSoldering -> Resistor_SMD:R_0402_1005Metric
- R31: renamed from R1; footprint pcb_v13:R_0805_HandSoldering -> Resistor_SMD:R_0402_1005Metric
- R4: renamed from R17; footprint pcb_v13:R_0805_HandSoldering -> Resistor_SMD:R_0402_1005Metric
- R5: renamed from R18; footprint pcb_v13:R_0805_HandSoldering -> Resistor_SMD:R_0402_1005Metric
- R7: renamed from R19; footprint pcb_v13:R_0805_HandSoldering -> Resistor_SMD:R_0402_1005Metric
- R8: renamed from R20; footprint pcb_v13:R_0805_HandSoldering -> Resistor_SMD:R_0402_1005Metric
- R9: renamed from R21; footprint pcb_v13:R_0805_HandSoldering -> Resistor_SMD:R_0402_1005Metric
- U10: renamed from U8; value 74LS257 -> 74HC257; footprint Housings_SSOP:SOP-16_4.4x10.4mm_Pitch1.27mm -> Package_SO:TSSOP-16_4.4x5mm_P0.65mm
- U11: renamed from U9; value 74LS257 -> 74HC257; footprint Housings_SSOP:SOP-16_4.4x10.4mm_Pitch1.27mm -> Package_SO:TSSOP-16_4.4x5mm_P0.65mm
- U3, U4: footprint Housings_SOIC:SOIC-20W_7.5x12.8mm_Pitch1.27mm -> Package_SO:TSSOP-20_4.4x6.5mm_P0.65mm
- U6: renamed from U1; value 74LS21 -> 74HC21
- U8: renamed from U6; value 74LS245 -> 74HC245; footprint Housings_SOIC:SOIC-20W_7.5x12.8mm_Pitch1.27mm -> Package_SO:TSSOP-20_4.4x6.5mm_P0.65mm
- U9: renamed from U7; value 74LS245 -> 74HC245; footprint Housings_SOIC:SOIC-20W_7.5x12.8mm_Pitch1.27mm -> Package_SO:TSSOP-20_4.4x6.5mm_P0.65mm
- renumbered D2 to D3, J3 to J2, J1 to J4, J2 to J5, U2 to U7
Connections:
- net +3V3: now also C10.1, C11.1, C12.1, C13.1, C14.1, C15.1, C18.1, C7.1, C8.1, C9.1, R14.1, U1.2 (VO), U2.1 (IOVDD), U2.10 (IOVDD), U2.22 (IOVDD), U2.33 (IOVDD), U2.42 (IOVDD), U2.43 (ADC_AVDD), U2.44 (VREG_IN), U2.48 (USB_VDD), U2.49 (IOVDD), U5.8 (VCC)
- net +5V: now also D2.2 (A); no longer C19.1, C20.2, C21.1, C22.1, C23.1, C24.1, D1.2 (A), D3.1 (K), R10.1, R11.1, R12.1, R13.1, R15.1, R22.1, R23.1, R24.1, R25.1, R26.1, R4.1, R5.1, R7.1, R8.1, R9.1, U10.16 (VCC), U11.16 (VCC), U6.14 (Vcc), U6.14 (Vcc), U7.14 (Vcc), U7.14 (Vcc), U7.14 (Vcc), U7.14 (Vcc), U8.1 (A->B), U8.20 (VCC), U9.1 (A->B), U9.20 (VCC)
- net GND: now also C1.2, C10.2, C11.2, C12.2, C13.2, C14.2, C15.2, C18.2, C2.2, C3.2, C4.2, C5.2, C6.2, C7.2, C8.2, C9.2, D4.3 (VSS), J1.5 (GND), J1.6 (Shield), J3.2 (Pin_2), U1.1 (GND), U2.19 (TESTEN), U2.57 (GND), U5.4 (GND); no longer U9.6 (A4)
- net SOL1: now also R35.1
- net SOL2: now also R34.1
- net SOL3: now also R33.1
- net SOL4: now also R32.1
- net TRIAC: now also R36.1
- net GPIO7: now reaches U3.11 (B8)
- net GPIO7: now also U2.9 (GPIO7)
- net GPIO6: now reaches U3.12 (B7)
- net GPIO6: now also U2.8 (GPIO6)
- net GPIO5: now reaches U3.13 (B6)
- net GPIO5: now also U2.7 (GPIO5)
- net GPIO4: now reaches U3.14 (B5)
- net GPIO4: now also U2.6 (GPIO4)
- net GPIO3: now reaches U3.15 (B4)
- net GPIO3: now also U2.5 (GPIO3)
- net GPIO2: now reaches U3.16 (B3)
- net GPIO2: now also U2.4 (GPIO2)
- net GPIO1: now reaches U3.17 (B2)
- net GPIO1: now also U2.3 (GPIO1)
- net GPIO0: now reaches U3.18 (B1)
- net GPIO0: now also U2.2 (GPIO0)
- net GPIO11: now reaches R16.2, U4.15 (B4)
- net GPIO11: now also U2.14 (GPIO11)
- net GPIO10: now reaches U4.16 (B3)
- net GPIO10: now also U2.13 (GPIO10)
- net GPIO9: now reaches U4.17 (B2)
- net GPIO9: now also U2.12 (GPIO9)
- net GPIO8: now reaches U4.18 (B1)
- net GPIO8: now also U2.11 (GPIO8)
- net GPIO12: now reaches TEST_MODE1.1 (Pin_1)
- net GPIO12: now also U2.15 (GPIO12)
- net GPIO14: now reaches R28.2, U9.5 (A3)
- net GPIO14: now also U2.17 (GPIO14)
- net GPIO15: now reaches U8.2 (A0)
- net GPIO15: now also U2.18 (GPIO15)
- net GPIO16: now reaches U8.3 (A1)
- net GPIO16: now also U2.27 (GPIO16)
- net GPIO17: now reaches U8.4 (A2)
- net GPIO17: now also U2.28 (GPIO17)
- net GPIO18: now reaches U8.5 (A3)
- net GPIO18: now also U2.29 (GPIO18)
- net GPIO19: now reaches U8.6 (A4)
- net GPIO19: now also U2.30 (GPIO19)
- net GPIO20: now reaches U8.7 (A5)
- net GPIO20: now also U2.31 (GPIO20)
- net GPIO21: now reaches U8.8 (A6)
- net GPIO21: now also U2.32 (GPIO21)
- net GPIO22: now reaches U8.9 (A7)
- net GPIO22: now also U2.34 (GPIO22)
- net GPIO26_ADC0: now reaches U9.2 (A0)
- net GPIO26_ADC0: now also U2.38 (GPIO26_ADC0)
- net GPIO27_ADC1: now reaches U9.3 (A1)
- net GPIO27_ADC1: now also U2.39 (GPIO27_ADC1)
- net GPIO28_ADC2: now reaches U9.4 (A2)
- net GPIO28_ADC2: now also U2.40 (GPIO28_ADC2)
- net at D1.1 (K): now also C4.1, D2.1 (K), U1.3 (VI)
- net PICO_WS2812: now reaches U9.14 (B4)
- net PICO_WS2812: now also D4.4 (DIN)
- net PICO_EN_OUT renamed GPIO13
- net GPIO13: now also U2.16 (GPIO13)
- new net: R2.2, U2.47 (USB_DP)
- new net: C2.1, R1.2, Y1.2
- new net: R3.2, U2.46 (USB_DM)
- new net +1V1: C3.1, C5.1, C6.1, U2.23 (DVDD), U2.45 (VREG_VOUT), U2.50 (DVDD)
- new net GPIO23: U2.35 (GPIO23), U9.6 (A4)
- new net GPIO24: U2.36 (GPIO24)
- new net GPIO25: U2.37 (GPIO25)
- new net GPIO29_ADC3: U2.41 (GPIO29_ADC3)
- new net QSPI_SCLK: U2.52 (QSPI_SCLK), U5.6 (CLK)
- new net QSPI_SD0: U2.53 (QSPI_SD0), U5.5 (DI(IO0))
- new net QSPI_SD1: U2.55 (QSPI_SD1), U5.2 (DO(IO1))
- new net QSPI_SD2: U2.54 (QSPI_SD2), U5.3 (IO2)
- new net QSPI_SD3: U2.51 (QSPI_SD3), U5.7 (IO3)
- new net QSPI_SS: R14.2, R6.1, U2.56 (QSPI_SS), U5.1 (~{CS})
- new net RUN: U2.26 (RUN)
- new net SWCLK: U2.24 (SWCLK)
- new net SWD: U2.25 (SWD)
- new net USB_D+: J1.3 (D+), R2.1
- new net USB_D-: J1.2 (D-), R3.1
- new net VBUS: D1.2 (A), J1.1 (VBUS)
- new net VCC: C19.1, C20.2, C21.1, C22.1, C23.1, C24.1, D3.1 (K), D4.1 (VDD), R10.1, R11.1, R12.1, R13.1, R15.1, R22.1, R23.1, R24.1, R25.1, R26.1, R32.2, R33.2, R34.2, R35.2, R36.2, R4.1, R5.1, R7.1, R8.1, R9.1, U10.16 (VCC), U11.16 (VCC), U6.14 (Vcc), U6.14 (Vcc), U7.14 (Vcc), U7.14 (Vcc), U7.14 (Vcc), U7.14 (Vcc), U8.1 (A->B), U8.20 (VCC), U9.1 (A->B), U9.20 (VCC)
- new net XIN: C1.1, U2.20 (XIN), Y1.1
- new net XOUT: R1.1, U2.21 (XOUT)
- new net ~{USB_BOOT}: J3.1 (Pin_1), R6.2
- no-connect marks 20 -> 15
Other:
- note added: "74257 used over 74157 as this IC leaves the outputs at high impedance when OUT_SEL is low."
- note added: "Crystal"
- note added: "Flash"
- note added: "Make sure C6 is close to pin 45 of RP2040"
- note added: "Make sure C9 is close to pin 44 of RP2040"
- note added: "Make sure R2 and R3 are close to RP2040"
- note added: "Power"
- note added: "Pullup resistors make the inputs CMOS compatible (HC series)"
- note added: "Status LED"
- note added: "WPC Bus Input"
- note removed: "74LS TTL ICs used as they do not contain clamping diodes and cannot leak power from the input pins to the power rail."
- note removed: "74LS257 used over 74157 as this IC leaves the outputs at high impedance when OUT_SEL is low."
- moved on the sheet: C16, C17, C19, C20, C21, C22, C23, C24, D1, D3, J2, J4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

Commit message: Power routing
Parts:
- added PWR_LED2: LED, LED_SMD:LED_0402_1005Metric, symbol Device:LED
- added R37: 1k, Resistor_SMD:R_0402_1005Metric, symbol Device:R_Small
- added TP1, TP2: TestPoint, TestPoint:TestPoint_Pad_D1.5mm, symbol Connector:TestPoint
Connections:
- net COMB_EV: now also TP1.1
- net GND: now also PWR_LED2.1 (K)
- net GPIO25: now also R37.2
- net OUT_SEL: now also TP2.1
- new net: PWR_LED2.2 (A), R37.1
- no-connect marks 15 -> 14
Other:
- note added: "Status LEDs"
- note removed: "Status LED"
Changed lines of the file:
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@@
   (junction (at 353.695 116.84) (diameter 0) (color 0 0 0 0)
   )
+  (junction (at 386.715 189.865) (diameter 0) (color 0 0 0 0)
+  )
   (junction (at 144.145 57.15) (diameter 0) (color 0 0 0 0)
   )
@@
   (no_connect (at 212.725 114.3))
   (no_connect (at 231.775 172.72))
-  (no_connect (at 140.335 252.73))
   (no_connect (at 47.625 254))
   (no_connect (at 212.725 119.38))
@@
     (stroke (width 0) (type default) (color 0 0 0 0))
   )
+  (wire (pts (xy 210.185 197.485) (xy 212.09 197.485))
+    (stroke (width 0) (type default) (color 0 0 0 0))
+  )
   (wire (pts (xy 125.095 204.47) (xy 140.335 204.47))
     (stroke (width 0) (type default) (color 0 0 0 0))
@@
     (stroke (width 0) (type default) (color 0 0 0 0))
   )
+  (wire (pts (xy 386.715 189.865) (xy 392.43 189.865))
+    (stroke (width 0) (type default) (color 0 0 0 0))
+  )
   (wire (pts (xy 278.765 224.155) (xy 278.765 206.375))
     (stroke (width 0) (type default) (color 0 0 0 0))
@@
     (stroke (width 0) (type default) (color 0 0 0 0))
   )
+  (wire (pts (xy 217.17 197.485) (xy 220.98 197.485))
+    (stroke (width 0) (type default) (color 0 0 0 0))
+  )
   (wire (pts (xy 280.035 165.1) (xy 280.035 167.64))
     (stroke (width 0) (type default) (color 0 0 0 0))
@@
     (stroke (width 0) (type default) (color 0 0 0 0))
   )
-  (wire (pts (xy 381.635 189.865) (xy 384.175 189.865))
+  (wire (pts (xy 381.635 189.865) (xy 386.715 189.865))
     (stroke (width 0) (type default) (color 0 0 0 0))
   )
@@
     (effects (font (size 3.9878 3.9878)) (justify left bottom))
   )
-  (text "Status LED" (at 218.44 156.845 0)
+  (text "Status LEDs" (at 218.44 156.845 0)
     (effects (font (size 1.27 1.27)) (justify left bottom))
   )
@@
     (effects (font (size 1.27 1.27)) (justify right bottom))
   )
+  (label "GPIO25" (at 210.185 197.485 180)
+    (effects (font (size 1.27 1.27)) (justify right bottom))
+  )
   (label "5V_IN" (at 380.365 22.86 0)
     (effects (font (size 1.27 1.27)) (justify left bottom))
@@
     (effects (font (size 1.27 1.27)) (justify left bottom))
   )
-  (label "OUT_SEL" (at 384.175 189.865 0)
+  (label "OUT_SEL" (at 392.43 189.865 0)
     (effects (font (size 1.27 1.27)) (justify left bottom))
   )
@@
     (pin "1")
   )
+  (symbol (lib_id "Device:R_Small") (at 214.63 197.485 270) (unit 1)
+    (in_bom yes) (on_board yes)
+    (property "Reference" "R37" (id 0) (at 220.98 198.755 90)
+      (effects (font (size 1.27 1.27)) (justify right))
+    )
+    (property "Value" "1k" (id 1) (at 215.9 197.485 90)
+      (effects (font (size 1.27 1.27)) (justify right))
+    )
+    (property "Footprint" "Resistor_SMD:R_0402_1005Metric" (id 2) (at 214.63 197.485 0)
+      (effects (font (size 1.27 1.27)) hide)
+    )
+    (property "Datasheet" "~" (id 3) (at 214.63 197.485 0)
+      (effects (font (size 1.27 1.27)) hide)
+    )
+    (property "JLCPCB" "C17673" (id 4) (at 214.63 197.485 90)
+      (effects (font (size 1.27 1.27)) hide)
+    )
+    (pin "1")
+    (pin "2")
+  )
   (symbol (lib_id "Device:C") (at 187.325 143.51 0) (unit 1)
     (in_bom yes) (on_board yes)
@@
     (pin "2")
   )
+  (symbol (lib_id "Device:LED") (at 220.98 201.295 90) (unit 1)
+    (in_bom yes) (on_board yes)
+    (property "Reference" "PWR_LED2" (id 0) (at 223.9772 200.3044 90)
+      (effects (font (size 1.27 1.27)) (justify right))
+    )
+    (property "Value" "LED" (id 1) (at 223.9772 202.6158 90)
+      (effects (font (size 1.27 1.27)) (justify right))
+    )
+    (property "Footprint" "LED_SMD:LED_0402_1005Metric" (id 2) (at 220.98 201.295 0)
+      (effects (font (size 1.27 1.27)) hide)
+    )
+    (property "Datasheet" "~" (id 3) (at 220.98 201.295 0)
+      (effects (font (size 1.27 1.27)) hide)
+    )
+    (property "JLCPCB" "C434432" (id 4) (at 220.98 201.295 90)
+      (effects (font (size 1.27 1.27)) hide)
+    )
+    (pin "1")
+    (pin "2")
+  )
   (symbol (lib_id "power:+3V3") (at 95.25 53.975 0) (unit 1)
     (in_bom yes) (on_board yes)
@@
     (pin "3")
   )
+  (symbol (lib_id "Connector:TestPoint") (at 386.715 189.865 0) (unit 1)
+    (in_bom yes) (on_board yes) (fields_autoplaced)
+    (property "Reference" "TP2" (id 0) (at 388.112 185.7283 0)
+      (effects (font (size 1.27 1.27)) (justify left))
+    )
+    (property "Value" "TestPoint" (id 1) (at 388.112 188.2652 0)
+      (effects (font (size 1.27 1.27)) (justify left))
+    )
+    (property "Footprint" "TestPoint:TestPoint_Pad_D1.5mm" (id 2) (at 391.795 189.865 0)
+      (effects (font (size 1.27 1.27)) hide)
+    )
+    (property "Datasheet" "~" (id 3) (at 391.795 189.865 0)
+      (effects (font (size 1.27 1.27)) hide)
+    )
+    (pin "1")
+  )
   (symbol (lib_id "power:+1V1") (at 73.025 137.16 0) (unit 1)
     (in_bom yes) (on_board yes)
@@
     (pin "4")
   )
+  (symbol (lib_id "power:GND") (at 220.98 205.105 0) (unit 1)
+    (in_bom yes) (on_board yes)
+    (property "Reference" "#PWR046" (id 0) (at 220.98 211.455 0)
+      (effects (font (size 1.27 1.27)) hide)
+    )
+    (property "Value" "GND" (id 1) (at 224.79 206.375 0))
+    (property "Footprint" "" (id 2) (at 220.98 205.105 0)
+      (effects (font (size 1.27 1.27)) hide)
+    )
+    (property "Datasheet" "" (id 3) (at 220.98 205.105 0)
+      (effects (font (size 1.27 1.27)) hide)
+    )
+    (pin "1")
+  )
   (symbol (lib_id "Device:C") (at 141.605 143.51 0) (unit 1)
     (in_bom yes) (on_board yes)
@@
     (pin "2")
   )
+  (symbol (lib_id "Connector:TestPoint") (at 338.455 192.405 180) (unit 1)
+    (in_bom yes) (on_board yes) (fields_autoplaced)
+    (property "Reference" "TP1" (id 0) (at 339.852 194.8723 0)
+      (effects (font (size 1.27 1.27)) (justify right))
+    )
+    (property "Value" "TestPoint" (id 1) (at 339.852 197.4092 0)
+      (effects (font (size 1.27 1.27)) (justify right))
+    )
+    (property "Footprint" "TestPoint:TestPoint_Pad_D1.5mm" (id 2) (at 333.375 192.405 0)
+      (effects (font (size 1.27 1.27)) hide)
+    )
+    (property "Datasheet" "~" (id 3) (at 333.375 192.405 0)
+      (effects (font (size 1.27 1.27)) hide)
+    )
+    (pin "1")
+  )
   (symbol (lib_id "power:GND") (at 52.705 149.86 0) (unit 1)
     (in_bom yes) (on_board yes)
@@
       (reference "#PWR045") (unit 1) (value "GND") (footprint "")
     )
+    (path "/ac14b154-cd8a-47b0-a09f-dc2873dab655"
+      (reference "#PWR046") (unit 1) (value "GND") (footprint "")
+    )
     (path "/549073c7-0ad8-4a26-b9dc-712dc8f06119"
       (reference "C1") (unit 1) (value "27p") (footprint "Capacitor_SMD:C_0402_1005Metric")
@@
       (reference "PWR_LED1") (unit 1) (value "LED") (footprint "LED_SMD:LED_0402_1005Metric")
     )
+    (path "/3838b934-d573-4bb0-a0e6-21e6637f2dc0"
+      (reference "PWR_LED2") (unit 1) (value "LED") (footprint "LED_SMD:LED_0402_1005Metric")
+    )
     (path "/e1d64be7-9a66-460f-9241-349f14555d8d"
       (reference "R1") (unit 1) (value "1k") (footprint "Resistor_SMD:R_0402_1005Metric")
@@
       (reference "R36") (unit 1) (value "4.7k") (footprint "Resistor_SMD:R_0402_1005Metric")
     )
+    (path "/223ae605-40ba-4f7c-a182-8344cfd44bfb"
+      (reference "R37") (unit 1) (value "1k") (footprint "Resistor_SMD:R_0402_1005Metric")
+    )
     (path "/00000000-0000-0000-0000-000061c323ff"
       (reference "TEST_MODE1") (unit 1) (value "Conn_01x02") (footprint "Pin_Headers:Pin_Header_Straight_1x02_Pitch2.54mm")
     )
+    (path "/fdb85c53-00b1-46fa-98f4-15a55c21c41a"
+      (reference "TP1") (unit 1) (value "TestPoint") (footprint "TestPoint:TestPoint_Pad_D1.5mm")
+    )
+    (path "/6d852f8e-c3b1-4bd3-af14-ea641ec56590"
+      (reference "TP2") (unit 1) (value "TestPoint") (footprint "TestPoint:TestPoint_Pad_D1.5mm")
+    )
     (path "/69a2888f-3318-437f-85c8-2bd516b2507a"

Commit message: Boettn
Parts:
- removed J3: Conn_01x02, Connector_PinHeader_2.54mm:PinHeader_1x02_P2.54mm_Vertical, symbol Connector_Generic:Conn_01x02
- added SW1: SW_Push, Button_Switch_SMD:SW_SPST_B3U-1000P, symbol Switch:SW_Push
Connections:
- net GND: now also SW1.1
- net ~{USB_BOOT}: now also SW1.2
Changed lines of the file:
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@@
     (stroke (width 0) (type default) (color 0 0 0 0))
   )
-  (wire (pts (xy 162.56 250.825) (xy 163.83 250.825))
-    (stroke (width 0) (type default) (color 0 0 0 0))
-  )
   (wire (pts (xy 197.485 57.15) (xy 182.245 57.15))
     (stroke (width 0) (type default) (color 0 0 0 0))
@@
     (stroke (width 0) (type default) (color 0 0 0 0))
   )
+  (wire (pts (xy 151.13 248.285) (xy 151.13 250.19))
+    (stroke (width 0) (type default) (color 0 0 0 0))
+  )
   (wire (pts (xy 84.455 171.45) (xy 84.455 158.75))
     (stroke (width 0) (type default) (color 0 0 0 0))
@@
     (stroke (width 0) (type default) (color 0 0 0 0))
   )
+  (wire (pts (xy 152.4 248.285) (xy 151.13 248.285))
+    (stroke (width 0) (type default) (color 0 0 0 0))
+  )
   (wire (pts (xy 215.9 224.155) (xy 209.55 224.155))
     (stroke (width 0) (type default) (color 0 0 0 0))
@@
     (stroke (width 0) (type default) (color 0 0 0 0))
   )
-  (wire (pts (xy 163.83 250.825) (xy 163.83 252.095))
-    (stroke (width 0) (type default) (color 0 0 0 0))
-  )
   (wire (pts (xy 194.31 248.285) (xy 196.85 248.285))
     (stroke (width 0) (type default) (color 0 0 0 0))
@@
     (pin "1")
   )
+  (symbol (lib_id "Switch:SW_Push") (at 157.48 248.285 0) (unit 1)
+    (in_bom yes) (on_board yes) (fields_autoplaced)
+    (property "Reference" "SW1" (id 0) (at 157.48 241.6642 0))
+    (property "Value" "SW_Push" (id 1) (at 157.48 244.2011 0))
+    (property "Footprint" "Button_Switch_SMD:SW_SPST_B3U-1000P" (id 2) (at 157.48 243.205 0)
+      (effects (font (size 1.27 1.27)) hide)
+    )
+    (property "Datasheet" "~" (id 3) (at 157.48 243.205 0)
+      (effects (font (size 1.27 1.27)) hide)
+    )
+    (pin "1")
+    (pin "2")
+  )
   (symbol (lib_id "Device:R_Small") (at 214.63 197.485 270) (unit 1)
     (in_bom yes) (on_board yes)
@@
     (pin "2")
   )
-  (symbol (lib_id "power:GND") (at 163.83 252.095 0) (unit 1)
+  (symbol (lib_id "power:GND") (at 151.13 250.19 0) (unit 1)
     (in_bom yes) (on_board yes)
-    (property "Reference" "#PWR018" (id 0) (at 163.83 258.445 0)
+    (property "Reference" "#PWR018" (id 0) (at 151.13 256.54 0)
       (effects (font (size 1.27 1.27)) hide)
     )
-    (property "Value" "GND" (id 1) (at 163.957 256.4892 0))
-    (property "Footprint" "" (id 2) (at 163.83 252.095 0)
+    (property "Value" "GND" (id 1) (at 151.257 254.5842 0))
+    (property "Footprint" "" (id 2) (at 151.13 250.19 0)
       (effects (font (size 1.27 1.27)) hide)
     )
-    (property "Datasheet" "" (id 3) (at 163.83 252.095 0)
+    (property "Datasheet" "" (id 3) (at 151.13 250.19 0)
       (effects (font (size 1.27 1.27)) hide)
     )
@@
     (pin "1")
   )
-  (symbol (lib_id "Connector_Generic:Conn_01x02") (at 157.48 248.285 0) (mirror y) (unit 1)
-    (in_bom yes) (on_board yes)
-    (property "Reference" "J3" (id 0) (at 156.21 244.475 0))
-    (property "Value" "Conn_01x02" (id 1) (at 156.21 254.635 0))
-    (property "Footprint" "Connector_PinHeader_2.54mm:PinHeader_1x02_P2.54mm_Vertical" (id 2) (at 157.48 248.285 0)
-      (effects (font (size 1.27 1.27)) hide)
-    )
-    (property "Datasheet" "~" (id 3) (at 157.48 248.285 0)
-      (effects (font (size 1.27 1.27)) hide)
-    )
-    (pin "1")
-    (pin "2")
-  )
   (symbol (lib_id "Diode:BAT60A") (at 73.66 31.75 180) (unit 1)
     (in_bom yes) (on_board yes)
@@
       (reference "J2") (unit 1) (value "Conn_01x02_Male") (footprint "Connectors_Molex:Molex_KK-6410-02_02x2.54mm_Straight")
     )
-    (path "/a9649279-f729-403e-9460-c1e67061c0ad"
-      (reference "J3") (unit 1) (value "Conn_01x02") (footprint "Connector_PinHeader_2.54mm:PinHeader_1x02_P2.54mm_Vertical")
-    )
     (path "/00000000-0000-0000-0000-000061751c78"
       (reference "J4") (unit 1) (value "Conn_02x17_Odd_Even") (footprint "Pin_Headers:Pin_Header_Straight_2x17_Pitch2.54mm")
@@
       (reference "R37") (unit 1) (value "1k") (footprint "Resistor_SMD:R_0402_1005Metric")
     )
+    (path "/222ff30c-5b43-423b-b5fa-9c7e3cb3294c"
+      (reference "SW1") (unit 1) (value "SW_Push") (footprint "Button_Switch_SMD:SW_SPST_B3U-1000P")
+    )
     (path "/00000000-0000-0000-0000-000061c323ff"
