File: pcb_v13/afterglow_pico.kicad_sch (KiCad schematic)
At the start: 87 parts, among them J1 USB_B_Micro, J2 Conn_01x02_Male, J4 Conn_02x17_Odd_Even, J5 Conn_02x17_Odd_Even, SW1 SW_Push, U1 NCP1117-3.3_SOT223, U10 74HC257, U11 74HC257, U2 RP2040, U3 SN74LVC245AN, U4 SN74LVC245AN, U5 W25Q32JVSS, U6 74HC21, U7 7408, U8 74HC245, U9 74HC245, Y1 ABLS-12.000MHZ-B4-T

Commit message: Almost
Parts:
- D4: JLCPCB (none) -> C2761795
- SW1: JLCPCB (none) -> C231329
- U2: JLCPCB (none) -> C2040
- U5: JLCPCB (none) -> C82344
Changed lines of the file:
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@@
+      (effects (font (size 1.27 1.27)) hide)
+    )
+    (property "JLCPCB" "C231329" (id 4) (at 157.48 248.285 0)
       (effects (font (size 1.27 1.27)) hide)
     )
@@
       (effects (font (size 1.27 1.27)) (justify left top) hide)
     )
+    (property "JLCPCB" "C2761795" (id 4) (at 224.155 172.72 0)
+      (effects (font (size 1.27 1.27)) hide)
+    )
     (pin "1")
     (pin "2")
@@
     )
     (property "Datasheet" "" (id 3) (at 74.295 222.25 0)
+      (effects (font (size 1.27 1.27)) hide)
+    )
+    (property "JLCPCB" "C2040" (id 4) (at 93.345 222.25 0)
       (effects (font (size 1.27 1.27)) hide)
     )
@@
       (effects (font (size 1.27 1.27)) hide)
     )
+    (property "JLCPCB" "C82344" (id 4) (at 209.55 250.825 0)
+      (effects (font (size 1.27 1.27)) hide)
+    )

Commit message: Forgot a resistor
Parts:
- added R38: 220, Resistor_SMD:R_0402_1005Metric, symbol Device:R_Small
- C1, C2: JLCPCB (none) -> C107002
- C10, C11, C12, C13, C14, C15, C18, C3, C5, C8: JLCPCB (none) -> C131394
- C16, C17, C19, C20, C21, C22, C23, C24: JLCPCB C396718 -> C131394
- C4, C7: JLCPCB (none) -> C89189
- J1: JLCPCB (none) -> C505111
- R1, R6: JLCPCB (none) -> C106235
- R29: value 180 -> 1k; JLCPCB C25270 -> C106235
- R37: JLCPCB C17673 -> C106235
- U1: JLCPCB (none) -> C26537
- Y1: JLCPCB (none) -> C390753
Connections:
- net PICO_WS2812: now also R38.2; no longer D4.4 (DIN)
- new net: D4.4 (DIN), R38.1
Changed lines of the file:
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@@
     (stroke (width 0) (type default) (color 0 0 0 0))
   )
+  (wire (pts (xy 208.915 172.72) (xy 211.455 172.72))
+    (stroke (width 0) (type default) (color 0 0 0 0))
+  )
   (wire (pts (xy 299.085 54.61) (xy 292.735 54.61))
     (stroke (width 0) (type default) (color 0 0 0 0))
@@
     (effects (font (size 1.27 1.27)) (justify left bottom))
   )
-  (label "PICO_WS2812" (at 216.535 172.72 180)
+  (label "PICO_WS2812" (at 208.915 172.72 180)
     (effects (font (size 1.27 1.27)) (justify right bottom))
   )
@@
       (effects (font (size 1.27 1.27)) hide)
     )
-    (property "JLCPCB" "C396718" (id 4) (at 215.265 43.18 0)
+    (property "JLCPCB" "C131394" (id 4) (at 215.265 43.18 0)
       (effects (font (size 1.27 1.27)) hide)
     )
@@
       (effects (font (size 1.27 1.27)) hide)
     )
-    (property "JLCPCB" "C396718" (id 4) (at 215.265 92.71 0)
+    (property "JLCPCB" "C131394" (id 4) (at 215.265 92.71 0)
       (effects (font (size 1.27 1.27)) hide)
     )
@@
       (effects (font (size 1.27 1.27)) hide)
     )
-    (property "JLCPCB" "C396718" (id 4) (at 377.825 25.4 0)
+    (property "JLCPCB" "C131394" (id 4) (at 377.825 25.4 0)
       (effects (font (size 1.27 1.27)) hide)
     )
@@
       (effects (font (size 1.27 1.27)) hide)
     )
-    (property "JLCPCB" "C396718" (id 4) (at 377.825 63.5 0)
+    (property "JLCPCB" "C131394" (id 4) (at 377.825 63.5 0)
       (effects (font (size 1.27 1.27)) hide)
     )
@@
       (effects (font (size 1.27 1.27)) hide)
     )
-    (property "JLCPCB" "C396718" (id 4) (at 323.215 45.72 0)
+    (property "JLCPCB" "C131394" (id 4) (at 323.215 45.72 0)
       (effects (font (size 1.27 1.27)) hide)
     )
@@
       (effects (font (size 1.27 1.27)) hide)
     )
-    (property "JLCPCB" "C396718" (id 4) (at 329.565 101.6 0)
+    (property "JLCPCB" "C131394" (id 4) (at 329.565 101.6 0)
       (effects (font (size 1.27 1.27)) hide)
     )
@@
       (effects (font (size 1.27 1.27)) hide)
     )
-    (property "JLCPCB" "C396718" (id 4) (at 310.515 172.085 0)
+    (property "JLCPCB" "C131394" (id 4) (at 310.515 172.085 0)
       (effects (font (size 1.27 1.27)) hide)
     )
@@
       (effects (font (size 1.27 1.27)) hide)
     )
-    (property "JLCPCB" "C396718" (id 4) (at 380.365 178.435 0)
+    (property "JLCPCB" "C131394" (id 4) (at 380.365 178.435 0)
       (effects (font (size 1.27 1.27)) hide)
     )
@@
       (effects (font (size 1.27 1.27)) (justify left))
     )
-    (property "Value" "180" (id 1) (at 308.483 41.783 0)
+    (property "Value" "1k" (id 1) (at 308.483 41.783 0)
       (effects (font (size 1.27 1.27)) (justify left))
     )
@@
       (effects (font (size 1.27 1.27)) hide)
     )
-    (property "JLCPCB" "C25270" (id 4) (at 306.705 40.64 0)
+    (property "JLCPCB" "C106235" (id 4) (at 306.705 40.64 0)
       (effects (font (size 1.27 1.27)) hide)
     )
@@
       (effects (font (size 1.27 1.27)) hide)
     )
+    (property "JLCPCB" "C131394" (id 4) (at 52.705 143.51 0)
+      (effects (font (size 1.27 1.27)) hide)
+    )
     (pin "1")
     (pin "2")
@@
       (effects (font (size 1.27 1.27)) hide)
     )
-    (property "JLCPCB" "C17673" (id 4) (at 214.63 197.485 90)
+    (property "JLCPCB" "C106235" (id 4) (at 214.63 197.485 90)
       (effects (font (size 1.27 1.27)) hide)
     )
@@
       (effects (font (size 1.27 1.27)) hide)
     )
+    (property "JLCPCB" "C131394" (id 4) (at 187.325 143.51 0)
+      (effects (font (size 1.27 1.27)) hide)
+    )
     (pin "1")
     (pin "2")
@@
       (effects (font (size 1.27 1.27)) hide)
     )
+    (property "JLCPCB" "C131394" (id 4) (at 64.135 143.51 0)
+      (effects (font (size 1.27 1.27)) hide)
+    )
     (pin "1")
     (pin "2")
@@
       (effects (font (size 1.27 1.27)) hide)
     )
+    (property "JLCPCB" "C131394" (id 4) (at 164.465 143.51 0)
+      (effects (font (size 1.27 1.27)) hide)
+    )
+    (pin "1")
+    (pin "2")
+  )
+  (symbol (lib_id "Device:R_Small") (at 213.995 172.72 270) (unit 1)
+    (in_bom yes) (on_board yes)
+    (property "Reference" "R38" (id 0) (at 220.345 173.99 90)
+      (effects (font (size 1.27 1.27)) (justify right))
+    )
+    (property "Value" "220" (id 1) (at 215.265 172.72 90)
+      (effects (font (size 1.27 1.27)) (justify right))
+    )
+    (property "Footprint" "Resistor_SMD:R_0402_1005Metric" (id 2) (at 213.995 172.72 0)
+      (effects (font (size 1.27 1.27)) hide)
+    )
+    (property "Datasheet" "~" (id 3) (at 213.995 172.72 0)
+      (effects (font (size 1.27 1.27)) hide)
+    )
+    (property "JLCPCB" "C227335" (id 4) (at 213.995 172.72 90)
+      (effects (font (size 1.27 1.27)) hide)
+    )
     (pin "1")
     (pin "2")
@@
       (effects (font (size 1.27 1.27)) hide)
     )
+    (property "JLCPCB" "C390753" (id 4) (at 52.07 111.125 90)
+      (effects (font (size 1.27 1.27)) hide)
+    )
     (pin "1")
     (pin "2")
@@
       (effects (font (size 1.27 1.27)) hide)
     )
+    (property "JLCPCB" "C131394" (id 4) (at 130.175 143.51 0)
+      (effects (font (size 1.27 1.27)) hide)
+    )
     (pin "1")
     (pin "2")
@@
       (effects (font (size 1.27 1.27)) hide)
     )
+    (property "JLCPCB" "C107002" (id 4) (at 36.83 106.045 0)
+      (effects (font (size 1.27 1.27)) hide)
+    )
     (pin "1")
     (pin "2")
@@
       (effects (font (size 1.27 1.27)) hide)
     )
+    (property "JLCPCB" "C131394" (id 4) (at 215.9 229.235 0)
+      (effects (font (size 1.27 1.27)) hide)
+    )
     (pin "1")
     (pin "2")
@@
       (effects (font (size 1.27 1.27)) hide)
     )
+    (property "JLCPCB" "C26537" (id 4) (at 77.47 55.245 0)
+      (effects (font (size 1.27 1.27)) hide)
+    )
     (pin "1")
     (pin "2")
@@
       (effects (font (size 1.27 1.27)) hide)
     )
+    (property "JLCPCB" "C505111" (id 4) (at 34.29 60.325 0)
+      (effects (font (size 1.27 1.27)) hide)
+    )
     (pin "1")
     (pin "2")
@@
       (effects (font (size 1.27 1.27)) hide)
     )
+    (property "JLCPCB" "C107002" (id 4) (at 36.83 116.205 0)
+      (effects (font (size 1.27 1.27)) hide)
+    )
     (pin "1")
     (pin "2")
@@
       (effects (font (size 1.27 1.27)) hide)
     )
+    (property "JLCPCB" "C89189" (id 4) (at 95.25 60.325 0)
+      (effects (font (size 1.27 1.27)) hide)
+    )
     (pin "1")
     (pin "2")
@@
       (effects (font (size 1.27 1.27)) hide)
     )
+    (property "JLCPCB" "C131394" (id 4) (at 141.605 143.51 0)
+      (effects (font (size 1.27 1.27)) hide)
+    )
     (pin "1")
     (pin "2")
@@
       (effects (font (size 1.27 1.27)) hide)
     )
+    (property "JLCPCB" "C131394" (id 4) (at 118.745 143.51 0)
+      (effects (font (size 1.27 1.27)) hide)
+    )
     (pin "1")
     (pin "2")
@@
       (effects (font (size 1.27 1.27)) hide)
     )
+    (property "JLCPCB" "C131394" (id 4) (at 153.035 143.51 0)
+      (effects (font (size 1.27 1.27)) hide)
+    )
     (pin "1")
     (pin "2")
@@
       (effects (font (size 1.27 1.27)) hide)
     )
+    (property "JLCPCB" "C106235" (id 4) (at 69.85 116.205 90)
+      (effects (font (size 1.27 1.27)) hide)
+    )
     (pin "1")
     (pin "2")
@@
       (effects (font (size 1.27 1.27)) hide)
     )
+    (property "JLCPCB" "C131394" (id 4) (at 175.895 143.51 0)
+      (effects (font (size 1.27 1.27)) hide)
+    )
     (pin "1")
     (pin "2")
@@
       (effects (font (size 1.27 1.27)) hide)
     )
+    (property "JLCPCB" "C106235" (id 4) (at 179.07 248.285 90)
+      (effects (font (size 1.27 1.27)) hide)
+    )
     (pin "1")
     (pin "2")
@@
       (effects (font (size 1.27 1.27)) hide)
     )
+    (property "JLCPCB" "C89189" (id 4) (at 64.135 60.325 0)
+      (effects (font (size 1.27 1.27)) hide)
+    )
     (pin "1")
     (pin "2")
@@
     )
     (path "/00000000-0000-0000-0000-000061b0b124"
-      (reference "R29") (unit 1) (value "180") (footprint "Resistor_SMD:R_0402_1005Metric")
+      (reference "R29") (unit 1) (value "1k") (footprint "Resistor_SMD:R_0402_1005Metric")
     )
     (path "/00000000-0000-0000-0000-0000618eae63"
@@
       (reference "R37") (unit 1) (value "1k") (footprint "Resistor_SMD:R_0402_1005Metric")
     )
+    (path "/2cfbcd58-006c-4114-901d-858c49f4d742"
+      (reference "R38") (unit 1) (value "220") (footprint "Resistor_SMD:R_0402_1005Metric")
+    )
     (path "/222ff30c-5b43-423b-b5fa-9c7e3cb3294c"

Commit message: JLCPCB part numbers
Parts:
- C6, C9: JLCPCB (none) -> C326568
- J5: JLCPCB (none) -> C18417
- PWR_LED1: JLCPCB C434432 -> C2898985
- PWR_LED2: JLCPCB C434432 -> C130719
- R10, R11, R12, R4, R5, R7, R8, R9: JLCPCB C17710 -> C114877
- R13: JLCPCB C4310 -> C114759
- R14: JLCPCB (none) -> C60489
- R15: JLCPCB C17772 -> C137847
- R16, R22, R23, R24, R25, R26, R27, R28, R30, R31, R32, R33, R34, R35, R36: JLCPCB C17673 -> C105871
- R17, R18, R19, R20, R21: JLCPCB C17477 -> C138289
- R2, R3: JLCPCB (none) -> C137890
- TEST_MODE1: JLCPCB (none) -> C124375
- U10, U11: JLCPCB C7754 -> C7646
- U3, U4: JLCPCB C6080 -> C6082
- U8, U9: JLCPCB C129580 -> C6779
