File: pcb_v13/afterglow_pico.kicad_sch (KiCad schematic)
At the start: 92 parts, among them J1 USB_B_Micro, J2 Conn_01x02_Male, J4 Conn_02x17_Odd_Even, J5 Conn_02x17_Odd_Even, SW1 SW_Push, U1 NCP1117-3.3_SOT223, U10 74HC257, U11 74HC257, U2 RP2040, U3 SN74LVC245AN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

Commit message: added some comments
Parts:
- removed D5, D6: 1N4148, Diode_SMD:D_SOD-523, symbol Diode:1N4148
- removed R39: 4.7k, Resistor_SMD:R_0402_1005Metric, symbol Device:R
- removed TP3: TestPoint, TestPoint:TestPoint_Pad_D1.5mm, symbol Connector:TestPoint
- J2: footprint Connector_Molex:Molex_KK-254_AE-6410-02A_1x02_P2.54mm_Vertical -> Connectors_Molex:Molex_KK-6410-02_02x2.54mm_Straight
- J4: footprint Connector_PinHeader_2.54mm:PinHeader_2x17_P2.54mm_Vertical -> Pin_Headers:Pin_Header_Straight_2x17_Pitch2.54mm
- J5: footprint Connector_PinHeader_2.54mm:PinHeader_2x17_P2.54mm_Vertical -> Pin_Headers:Pin_Header_Straight_2x17_Pitch2.54mm; JLCPCB C2894978 -> C18417
- PWR_LED1: renamed from PWR1; JLCPCB C434449 -> C2898985
- R17, R18, R20, R21: JLCPCB (none) -> C138289
- TEST_MODE1: footprint Connector_PinHeader_2.54mm:PinHeader_1x02_P2.54mm_Vertical -> Pin_Headers:Pin_Header_Straight_1x02_Pitch2.54mm
- U6, U7: footprint Package_SO:SOIC-14_3.9x8.7mm_P1.27mm -> Housings_SOIC:SOIC-14_3.9x8.7mm_Pitch1.27mm
- U8, U9: value 74HCT245 -> 74HC245
Connections:
- net +3V3: now also R27.2
- net GND: now also U9.7 (A5)
- net GPIO13: now also R27.1, U10.15 (~{EN}), U11.15 (~{EN}); no longer U9.7 (A5)
- net VCC: no longer R27.2
- now unconnected: U9.13 (B5)
- no-connect marks 13 -> 14
Other:
- note added: "SW ROW 1/2 and SW COL 1/2 are input lines from Left and right flippers, no need so handle them. SW J1/2 go to jumpers and the line level ciruitry and appear to be unused."
- note removed: "Pullup to the 5V rail ensures pullup even when 3.3V is not powered"
- moved on the sheet: R27

Commit message: Restored lost PCB v1.3 schematic
Parts:
- added D5, D6: 1N4148, Diode_SMD:D_SOD-523, symbol Diode:1N4148
- added R39: 4.7k, Resistor_SMD:R_0402_1005Metric, symbol Device:R
- added TP3: TestPoint, TestPoint:TestPoint_Pad_D1.5mm, symbol Connector:TestPoint
- J2: footprint Connectors_Molex:Molex_KK-6410-02_02x2.54mm_Straight -> Connector_Molex:Molex_KK-254_AE-6410-02A_1x02_P2.54mm_Vertical
- J4: footprint Pin_Headers:Pin_Header_Straight_2x17_Pitch2.54mm -> Connector_PinHeader_2.54mm:PinHeader_2x17_P2.54mm_Vertical
- J5: footprint Pin_Headers:Pin_Header_Straight_2x17_Pitch2.54mm -> Connector_PinHeader_2.54mm:PinHeader_2x17_P2.54mm_Vertical; JLCPCB C18417 -> C2894978
- PWR1: renamed from PWR_LED1; JLCPCB C2898985 -> C434449
- R17, R18, R20, R21: JLCPCB C138289 -> (none)
- TEST_MODE1: footprint Pin_Headers:Pin_Header_Straight_1x02_Pitch2.54mm -> Connector_PinHeader_2.54mm:PinHeader_1x02_P2.54mm_Vertical
- U6, U7: footprint Housings_SOIC:SOIC-14_3.9x8.7mm_Pitch1.27mm -> Package_SO:SOIC-14_3.9x8.7mm_P1.27mm
- U8, U9: value 74HC245 -> 74HCT245
Connections:
- net +3V3: no longer R27.2
- net GND: no longer U9.7 (A5)
- net GPIO13: now also U9.7 (A5), D6.1 (K), TP3.1; no longer R27.1, U10.15 (~{EN}), U11.15 (~{EN})
- net VCC: now also R27.2, R39.1
- net at U9.13 (B5): now also U10.15 (~{EN}), U11.15 (~{EN}), R39.2
- new net: D5.2 (A), R27.1
- new net: D5.1 (K), D6.2 (A)
- no-connect marks 14 -> 13
Other:
- note added: "Pullup to the 5V rail ensures pullup even when 3.3V is not powered"
- note removed: "SW ROW 1/2 and SW COL 1/2 are input lines from Left and right flippers, no need so handle them. SW J1/2 go to jumpers and the line level ciruitry and appear to be unused."
- moved on the sheet: R27
