File: pcb_v13/afterglow_pico.kicad_sch (KiCad schematic)
At the start: 88 parts, among them J1 USB_B_Micro, J2 Conn_01x02_Male, J4 Conn_02x17_Odd_Even, J5 Conn_02x17_Odd_Even, SW1 SW_Push, U1 NCP1117-3.3_SOT223, U10 74HC257, U11 74HC257, U2 RP2040, U3 SN74LVC245AN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

Commit message: Minor corrections
Parts:
- U6: JLCPCB C2862597 -> C75398
- U6: JLCPCB (none) -> C75398
- U7: JLCPCB C6802 -> C5593
Changed lines of the file:
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@@
       (effects (font (size 1.27 1.27)) hide)
     )
-    (property "JLCPCB" "C2862597" (id 4) (at 296.545 183.515 0)
+    (property "JLCPCB" "C75398" (id 4) (at 296.545 183.515 0)
       (effects (font (size 1.27 1.27)) hide)
     )
@@
     )
     (property "Datasheet" "" (id 3) (at 296.545 202.565 0)
+      (effects (font (size 1.27 1.27)) hide)
+    )
+    (property "JLCPCB" "C75398" (id 4) (at 296.545 202.565 0)
       (effects (font (size 1.27 1.27)) hide)
     )
@@
       (effects (font (size 1.27 1.27)) hide)
     )
-    (property "JLCPCB" "C6802" (id 4) (at 324.485 192.405 0)
+    (property "JLCPCB" "C5593" (id 4) (at 324.485 192.405 0)
       (effects (font (size 1.27 1.27)) hide)
     )
@@
       (effects (font (size 1.27 1.27)) hide)
     )
-    (property "JLCPCB" "C6802" (id 4) (at 365.125 189.865 0)
+    (property "JLCPCB" "C5593" (id 4) (at 365.125 189.865 0)
       (effects (font (size 1.27 1.27)) hide)
     )
@@
       (effects (font (size 1.27 1.27)) hide)
     )
-    (property "JLCPCB" "C6802" (id 4) (at 296.545 219.075 0)
+    (property "JLCPCB" "C5593" (id 4) (at 296.545 219.075 0)
       (effects (font (size 1.27 1.27)) hide)
     )
@@
       (effects (font (size 1.27 1.27)) hide)
     )
-    (property "JLCPCB" "C6802" (id 4) (at 324.485 216.535 0)
-      (effects (font (size 1.27 1.27)) hide)
-    )
+    (property "JLCPCB" "C5593" (id 4) (at 324.485 216.535 0)
+      (effects (font (size 1.27 1.27)) hide)
+    )

Commit message: PCB v1.3b preparations
Parts:
- added D5, D6: 1N4148, Diode_SMD:D_SOD-523, symbol Diode:1N4148
- added R39: 4.7k, Resistor_SMD:R_0402_1005Metric, symbol Device:R
- added TP3: TestPoint, TestPoint:TestPoint_Pad_D1.5mm, symbol Connector:TestPoint
- J2: footprint Connectors_Molex:Molex_KK-6410-02_02x2.54mm_Straight -> Connector_Molex:Molex_KK-254_AE-6410-02A_1x02_P2.54mm_Vertical
- J4, J5: footprint Pin_Headers:Pin_Header_Straight_2x17_Pitch2.54mm -> Connector_PinHeader_2.54mm:PinHeader_2x17_P2.54mm_Vertical
- PWR: renamed from PWR_LED1; JLCPCB C2898985 -> C434449
- TEST_MODE1: footprint Pin_Headers:Pin_Header_Straight_1x02_Pitch2.54mm -> Connector_PinHeader_2.54mm:PinHeader_1x02_P2.54mm_Vertical
- U6, U7: footprint Housings_SOIC:SOIC-14_3.9x8.7mm_Pitch1.27mm -> Package_SO:SOIC-14_3.9x8.7mm_P1.27mm
- U8, U9: value 74HC245 -> 74HCT245
Connections:
- net +3V3: no longer R27.2
- net GND: no longer U9.7 (A5)
- net GPIO13: now also U9.7 (A5), D6.1 (K), TP3.1; no longer R27.1, U10.15 (~{EN}), U11.15 (~{EN})
- net VCC: now also R27.2, R39.1
- net at U9.13 (B5): now also U10.15 (~{EN}), U11.15 (~{EN}), R39.2
- new net: D5.2 (A), R27.1
- new net: D5.1 (K), D6.2 (A)
- no-connect marks 14 -> 13
Other:
- note added: "Pullup to the 5V rail ensures pullup even when 3.3V is not powered"
- moved on the sheet: R27

Commit message: PCB v1.3b
Parts:
- renumbered PWR to PWR1
Changed lines of the file:
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@@
   (symbol (lib_id "Device:LED") (at 306.705 48.26 90) (unit 1)
     (in_bom yes) (on_board yes) (dnp no)
-    (property "Reference" "PWR" (at 309.7022 47.2694 90)
+    (property "Reference" "PWR1" (at 309.7022 47.2694 90)
       (effects (font (size 1.27 1.27)) (justify right))
     )
@@
       (project "afterglow_pico"
         (path "/db36f6e3-e72a-487f-bda9-88cc84536f62"
-          (reference "PWR") (unit 1)
+          (reference "PWR1") (unit 1)
         )
       )

Commit message: PCB v1.3b touchup
Parts:
- J5: JLCPCB C18417 -> C2894978
Changed lines of the file:
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@@
       (effects (font (size 1.27 1.27)) hide)
     )
-    (property "JLCPCB" "C18417" (at 371.475 129.54 0)
+    (property "JLCPCB" "C2894978" (at 371.475 129.54 0)
       (effects (font (size 1.27 1.27)) hide)
     )

Commit message: Do not populate R17,R18,R20,R21
Parts:
- R17, R18, R20, R21: JLCPCB C138289 -> (none)
Changed lines of the file:
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@@
       (effects (font (size 1.27 1.27)) hide)
     )
-    (property "JLCPCB" "C138289" (at 269.875 221.615 90)
+    (property "JLCPCB" "" (at 269.875 221.615 90)
       (effects (font (size 1.27 1.27)) hide)
     )
@@
       (effects (font (size 1.27 1.27)) hide)
     )
-    (property "JLCPCB" "C138289" (at 269.875 216.535 90)
+    (property "JLCPCB" "" (at 269.875 216.535 90)
       (effects (font (size 1.27 1.27)) hide)
     )
@@
       (effects (font (size 1.27 1.27)) hide)
     )
-    (property "JLCPCB" "C138289" (at 269.875 201.295 90)
+    (property "JLCPCB" "" (at 269.875 201.295 90)
       (effects (font (size 1.27 1.27)) hide)
     )
@@
       (effects (font (size 1.27 1.27)) hide)
     )
-    (property "JLCPCB" "C138289" (at 269.875 203.835 90)
-      (effects (font (size 1.27 1.27)) hide)
-    )
+    (property "JLCPCB" "" (at 269.875 203.835 90)
+      (effects (font (size 1.27 1.27)) hide)
+    )
